File: hardware/usb-tester.sch (KiCad schematic (older format))
At the start: 13 parts

Commit message: Move symbols to 'ic' library
Parts:
- U?: symbol parts:STMPS2151STR -> ic:STMPS2151STR
- U?: symbol parts:FSUSB30MUX -> ic:FSUSB30MUX
Changed lines of the file:
@@
 Connection ~ 9600 1100
 $Comp
-L parts:STMPS2151STR U?
+L ic:STMPS2151STR U?
 U 1 1 5E3CBD43
 P 2000 5400
@@
 $EndComp
 $Comp
-L parts:FSUSB30MUX U?
+L ic:FSUSB30MUX U?
 U 1 1 5E3CC2D2
 P 6150 5150

Commit message: Muxes
Parts:
- added J?: Conn_01x03_Male, symbol Connector:Conn_01x03_Male
- added U? (x2): CD74HC4067SM, Package_SO:SSOP-24_5.3x8.2mm_P0.65mm, symbol 74xx:CD74HC4067SM
- added U? (x6): FSUSB30MUX, Package_SO:MSOP-10_3x3mm_P0.5mm, symbol ic:FSUSB30MUX
- added U?: 4514, symbol 4xxx_IEEE:4514
Connections:
- net T0_RX is gone; now on net T_RX: J?.10 (Pin_10)
- net T0_USB_DM is gone; now on net T_USB_DM0: J?.1 (Pin_1)
- net T0_USB_DP is gone; now on net T_USB_DP0: J?.2 (Pin_2)
- net +3V3: now also U?.10 (VCC), U?.1 (EL), U?.10 (VCC), U?.10 (VCC), U?.10 (VCC), U?.10 (VCC), U?.10 (VCC), U?.10 (VCC), U?.24 (VCC), U?.24 (VCC), U?.24 (Vdd)
- net GND: now also U?.12 (GND), U?.12 (GND), U?.12 (Vss), U?.13 (S3), U?.13 (S3), U?.22 (A3), U?.5 (GND), U?.5 (GND), U?.5 (GND)
- net SWDIO: now also U?.1 (COM); no longer J?.7 (Pin_7)
- net T_NRST: no longer J?.5 (Pin_5)
- net T_TX: now also U?.1 (COM)
- net USBT_DM: now also U?.6 (D-)
- net USBT_DP: now also U?.4 (D+)
- net SEL0: now reaches U?.1 (S)
- net SEL0: now also U?.1 (S), U?.1 (S), U?.1 (S), U?.10 (S0), U?.10 (S0), U?.2 (A0)
- net T_USB_DP0: now reaches U?.2 (HSD1+)
- net T_USB_DP1: now reaches U?.3 (HSD2+)
- net A_DP0: now reaches U?.4 (D+)
- net A_DP0: now also U?.2 (HSD1+)
- net at U?.5 (GND): now also U?.5 (GND), U?.5 (GND), U?.5 (GND)
- net A_DM0: now reaches U?.6 (D-)
- net A_DM0: now also U?.8 (HSD1-)
- net T_USB_DM1: now reaches U?.7 (HSD2-)
- net T_USB_DM0: now reaches U?.8 (HSD1-)
- net MUXEN: now reaches U?.9 (~OE)
- net MUXEN: now also U?.15 (~E), U?.15 (~E), U?.9 (~OE), U?.9 (~OE), U?.9 (~OE), U?.9 (~OE), U?.9 (~OE), U?.9 (~OE)
- net T0_TX renamed T_TX0
- net T_TX0: now also U?.9 (I0)
- new net A_DM1: U?.6 (D-), U?.7 (HSD2-)
- new net A_DM2: U?.6 (D-), U?.8 (HSD1-)
- new net A_DM3: U?.6 (D-), U?.7 (HSD2-)
- new net A_DP1: U?.3 (HSD2+), U?.4 (D+)
- new net A_DP2: U?.2 (HSD1+), U?.4 (D+)
- new net A_DP3: U?.3 (HSD2+), U?.4 (D+)
- new net B_DM0: U?.6 (D-), U?.8 (HSD1-)
- new net B_DM1: U?.6 (D-), U?.7 (HSD2-)
- new net B_DP0: U?.2 (HSD1+), U?.4 (D+)
- new net B_DP1: U?.3 (HSD2+), U?.4 (D+)
- new net SEL1: U?.1 (S), U?.1 (S), U?.11 (S1), U?.11 (S1), U?.3 (A1)
- new net SEL2: U?.1 (S), U?.14 (S2), U?.14 (S2), U?.21 (A2)
- new net T_NRST0: J?.5 (Pin_5), U?.11 (Q0)
- new net T_NRST1: U?.9 (Q1)
- new net T_NRST2: U?.10 (Q2)
- new net T_NRST3: U?.8 (Q3)
- new net T_NRST4: U?.7 (Q4)
- new net T_NRST5: U?.6 (Q5)
- new net T_NRST6: U?.5 (Q6)
- new net T_NRST7: U?.4 (Q7)
- new net T_RST: U?.23 (~EN)
- new net T_SWDIO0: J?.7 (Pin_7), U?.9 (I0)
- new net T_SWDIO1: U?.8 (I1)
- new net T_SWDIO2: U?.7 (I2)
- new net T_SWDIO3: U?.6 (I3)
- new net T_SWDIO4: U?.5 (I4)
- new net T_SWDIO5: U?.4 (I5)
- new net T_SWDIO6: U?.3 (I6)
- new net T_SWDIO7: U?.2 (I7)
- new net T_TX1: U?.8 (I1)
- new net T_TX2: U?.7 (I2)
- new net T_TX3: U?.6 (I3)
- new net T_TX4: U?.5 (I4)
- new net T_TX5: U?.4 (I5)
- new net T_TX6: U?.3 (I6)
- new net T_TX7: U?.2 (I7)
- new net T_USB_DM2: U?.8 (HSD1-)
- new net T_USB_DM3: U?.7 (HSD2-)
- new net T_USB_DM4: U?.8 (HSD1-)
- new net T_USB_DM5: U?.7 (HSD2-)
- new net T_USB_DM6: U?.8 (HSD1-)
- new net T_USB_DM7: U?.7 (HSD2-)
- new net T_USB_DP2: U?.2 (HSD1+)
- new net T_USB_DP3: U?.3 (HSD2+)
- new net T_USB_DP4: U?.2 (HSD1+)
- new net T_USB_DP5: U?.3 (HSD2+)
- new net T_USB_DP6: U?.2 (HSD1+)
- new net T_USB_DP7: U?.3 (HSD2+)
- no-connect marks 7 -> 31
Other:
- moved on the sheet: C?, J?, U?

Commit message: Base board
Parts:
- removed J?: TEST, symbol Connector:USB_B_Micro
- removed SW?: NEXT, symbol Switch:SW_SPST
- removed U?: STM32F042F6Px, Package_SO:TSSOP-20_4.4x6.5mm_P0.65mm, symbol MCU_ST_STM32F0:STM32F042F6Px
- removed U?: USBLC6-2SC6, Package_TO_SOT_SMD:SOT-23-6, symbol Power_Protection:USBLC6-2SC6
- removed U? (x5): FSUSB30MUX, Package_SO:MSOP-10_3x3mm_P0.5mm, symbol ic:FSUSB30MUX
- added J?: Upstream, symbol Connector:Conn_01x03_Male
- added J? (x3): Target1, symbol Connector:Conn_01x03_Male
- added J?: Target 1, symbol Connector_Generic:Conn_02x05_Odd_Even
- added J?: Target 2, symbol Connector_Generic:Conn_02x05_Odd_Even
- added J?: Target 3, symbol Connector_Generic:Conn_02x05_Odd_Even
- added J?: Comm, symbol Connector:Conn_01x05_Male
- added J?: STDC14, symbol Connector_Generic:Conn_02x07_Odd_Even
- J?: value PROGRAM -> TARGET
- J?: value Conn_01x03_Male -> Target0
Connections:
- net A_DM0 is gone; now on net USB_DM: U?.6 (D-)
- net A_DM1 is gone; now on net USB_DM: U?.6 (D-)
- net A_DP0 is gone; now on net USB_DP: U?.4 (D+)
- net A_DP1 is gone; now on net USB_DP: U?.4 (D+)
- net SEL2 is gone; now on net GND: U?.14 (S2), U?.14 (S2), U?.21 (A2)
- net T_RST is gone; now on net GND: U?.23 (~EN)
- net GND: now also J?.3 (Pin_3), U?.5 (GND), U?.5 (GND), J?.1 (Pin_1), J?.11 (Pin_11), J?.3 (Pin_3), J?.3 (Pin_3), J?.3 (Pin_3), J?.3 (Pin_3), J?.4 (Pin_4), J?.4 (Pin_4), J?.4 (Pin_4), J?.5 (Pin_5), J?.7 (Pin_7); no longer U?.22 (A3)
- net MUXEN: no longer U?.9 (~OE), U?.9 (~OE)
- net SWCLK: now also J?.6 (Pin_6), J?.8 (Pin_8), J?.8 (Pin_8), J?.8 (Pin_8)
- net SWDIO: now also J?.4 (Pin_4)
- net T_CLK: now also J?.2 (Pin_2), J?.6 (Pin_6), J?.6 (Pin_6), J?.6 (Pin_6)
- net T_NRST: now also U?.22 (A3), J?.12 (Pin_12), J?.3 (Pin_3)
- net T_NRST0: now also U?.18 (Q8); no longer U?.11 (Q0)
- net T_NRST1: now also U?.17 (Q9), J?.5 (Pin_5); no longer U?.9 (Q1)
- net T_NRST2: now also U?.20 (Q10), J?.5 (Pin_5); no longer U?.10 (Q2)
- net T_NRST3: now also U?.19 (Q11), J?.5 (Pin_5); no longer U?.8 (Q3)
- net T_RX: now also J?.10 (Pin_10), J?.10 (Pin_10), J?.10 (Pin_10), J?.13 (Pin_13), J?.5 (Pin_5)
- net T_SWDIO1: now also J?.7 (Pin_7)
- net T_SWDIO2: now also J?.7 (Pin_7)
- net T_SWDIO3: now also J?.7 (Pin_7)
- net T_TX: now also J?.14 (Pin_14), J?.4 (Pin_4)
- net T_TX1: now also J?.9 (Pin_9)
- net T_TX2: now also J?.9 (Pin_9)
- net T_TX3: now also J?.9 (Pin_9)
- net T_USB_DM0: now also J?.2 (Pin_2)
- net T_USB_DM1: now also J?.1 (Pin_1), J?.2 (Pin_2)
- net T_USB_DM2: now also J?.1 (Pin_1), J?.2 (Pin_2)
- net T_USB_DM3: now also J?.1 (Pin_1), J?.2 (Pin_2)
- net T_USB_DP0: now also J?.1 (Pin_1)
- net T_USB_DP1: now also J?.1 (Pin_1), J?.2 (Pin_2)
- net T_USB_DP2: now also J?.1 (Pin_1), J?.2 (Pin_2)
- net T_USB_DP3: now also J?.1 (Pin_1), J?.2 (Pin_2)
- net T_VCC: now also J?.3 (Pin_3), J?.3 (Pin_3), J?.3 (Pin_3), J?.3 (Pin_3)
- net USB_DM: now also J?.2 (Pin_2)
- net USB_DP: now also J?.1 (Pin_1)
- net T_NRST4: no longer names the net of U?.7 (Q4)
- net T_NRST5: no longer names the net of U?.6 (Q5)
- net T_NRST6: no longer names the net of U?.5 (Q6)
- net T_NRST7: no longer names the net of U?.4 (Q7)
- net T_SWDIO4: no longer names the net of U?.5 (I4)
- net T_SWDIO5: no longer names the net of U?.4 (I5)
- net T_SWDIO6: no longer names the net of U?.3 (I6)
- net T_SWDIO7: no longer names the net of U?.2 (I7)
- net T_TX4: no longer names the net of U?.5 (I4)
- net T_TX5: no longer names the net of U?.4 (I5)
- net T_TX6: no longer names the net of U?.3 (I6)
- net T_TX7: no longer names the net of U?.2 (I7)
- new net USBMUXEN0: U?.9 (~OE)
- new net USBMUXEN1: U?.9 (~OE)
- no-connect marks 31 -> 46
Other:
- moved on the sheet: J?, U?

Commit message: Updated connectors and labels on the main board
Parts:
- removed J?: Comm, symbol Connector:Conn_01x05_Male
- added J11: Comm, symbol Connector:Conn_01x10_Male
- added J?: SWD, symbol Connector:Conn_01x06_Male
- added J?: UART, symbol Connector:Conn_01x02_Male
- gave numbers to parts that had none: 22
Connections:
- net T_CLK is gone; now on net GND: J2.6 (Pin_6), J3.6 (Pin_6), J4.6 (Pin_6), J5.6 (Pin_6)
- net GND: now also J11.1 (Pin_1), J?.3 (Pin_3); no longer J2.4 (Pin_4), J3.4 (Pin_4), J4.4 (Pin_4), J5.4 (Pin_4)
- net PWR_EN: now also J11.10 (Pin_10)
- net SEL0: now also J11.6 (Pin_6)
- net SEL1: now also J11.7 (Pin_7)
- net SWCLK: now also J2.10 (Pin_10), J3.10 (Pin_10), J4.10 (Pin_10), J5.10 (Pin_10), J?.2 (Pin_2); no longer J2.8 (Pin_8), J3.8 (Pin_8), J4.8 (Pin_8), J5.8 (Pin_8)
- net SWDIO: now also J?.4 (Pin_4)
- net T_NRST: now also J11.3 (Pin_3), J?.5 (Pin_5)
- net T_RX: now also J2.3 (Pin_3), J3.3 (Pin_3), J4.3 (Pin_3), J5.3 (Pin_3), J11.5 (Pin_5), J?.1 (Pin_1); no longer J2.10 (Pin_10), J3.10 (Pin_10), J4.10 (Pin_10), J5.10 (Pin_10)
- net T_TX: now also J11.4 (Pin_4), J?.2 (Pin_2)
- net T_VCC: now also J2.8 (Pin_8), J3.8 (Pin_8), J4.8 (Pin_8), J5.8 (Pin_8), J?.1 (Pin_1); no longer J2.3 (Pin_3), J3.3 (Pin_3), J4.3 (Pin_3), J5.3 (Pin_3)
- net USBMUXEN0: now also J11.8 (Pin_8)
- net USBMUXEN1: now also J11.9 (Pin_9)
- net T_NRST0 renamed T0_NRST
- net T0_NRST: now also J2.1 (Pin_1); no longer J2.5 (Pin_5)
- net T_NRST1 renamed T1_NRST
- net T1_NRST: now also J3.1 (Pin_1); no longer J3.5 (Pin_5)
- net T_NRST2 renamed T2_NRST
- net T2_NRST: now also J4.1 (Pin_1); no longer J4.5 (Pin_5)
- net T_NRST3 renamed T3_NRST
- net T3_NRST: now also J5.1 (Pin_1); no longer J5.5 (Pin_5)
- net T_SWDIO0 renamed T0_SWDIO
- net T0_SWDIO: now also J2.9 (Pin_9); no longer J2.7 (Pin_7)
- net T_SWDIO1 renamed T1_SWDIO
- net T1_SWDIO: now also J3.9 (Pin_9); no longer J3.7 (Pin_7)
- net T_SWDIO2 renamed T2_SWDIO
- net T2_SWDIO: now also J4.9 (Pin_9); no longer J4.7 (Pin_7)
- net T_SWDIO3 renamed T3_SWDIO
- net T3_SWDIO: now also J5.9 (Pin_9); no longer J5.7 (Pin_7)
- net T_TX0 renamed T0_TX
- net T0_TX: now also J2.4 (Pin_4); no longer J2.9 (Pin_9)
- net T_TX1 renamed T1_TX
- net T1_TX: now also J3.4 (Pin_4); no longer J3.9 (Pin_9)
- net T_TX2 renamed T2_TX
- net T2_TX: now also J4.4 (Pin_4); no longer J4.9 (Pin_9)
- net T_TX3 renamed T3_TX
- net T3_TX: now also J5.4 (Pin_4); no longer J5.9 (Pin_9)
- net T_USB_DM0 renamed T0_USB_D-
- net T0_USB_D-: now also J2.5 (Pin_5); no longer J2.1 (Pin_1)
- net T_USB_DM1 renamed T1_USB_D-
- net T1_USB_D-: now also J3.5 (Pin_5); no longer J3.1 (Pin_1)
- net T_USB_DM2 renamed T2_USB_D-
- net T2_USB_D-: now also J4.5 (Pin_5); no longer J4.1 (Pin_1)
- net T_USB_DM3 renamed T3_USB_D-
- net T3_USB_D-: now also J5.5 (Pin_5); no longer J5.1 (Pin_1)
- net T_USB_DP0 renamed T0_USB_D+
- net T0_USB_D+: now also J2.7 (Pin_7); no longer J2.2 (Pin_2)
- net T_USB_DP1 renamed T1_USB_D+
- net T1_USB_D+: now also J3.7 (Pin_7); no longer J3.2 (Pin_2)
- net T_USB_DP2 renamed T2_USB_D+
- net T2_USB_D+: now also J4.7 (Pin_7); no longer J4.2 (Pin_2)
- net T_USB_DP3 renamed T3_USB_D+
- net T3_USB_D+: now also J5.7 (Pin_7); no longer J5.2 (Pin_2)
- net USB_DM renamed USB_D-
- net USB_DP renamed USB_D+
- new net T_BOOT0: J11.2 (Pin_2), J2.2 (Pin_2), J3.2 (Pin_2), J4.2 (Pin_2), J5.2 (Pin_2)
Other:
- moved on the sheet: J12

Commit message: Main board schematic
Parts:
- removed J1: STDC14, symbol Connector_Generic:Conn_02x07_Odd_Even
- removed J11: Comm, symbol Connector:Conn_01x10_Male
- removed J12: SWD, symbol Connector:Conn_ARM_JTAG_SWD_10
- removed J?: SWD, symbol Connector:Conn_01x06_Male
- removed J?: UART, symbol Connector:Conn_01x02_Male
- removed U7: CD74HC4067SM, Package_SO:SSOP-24_5.3x8.2mm_P0.65mm, symbol 74xx:CD74HC4067SM
- added J12: SWD2, Connector_PinHeader_2.54mm:PinHeader_1x03_P2.54mm_Vertical, symbol Connector:Conn_01x03_Male
- added J15: SWD3, Connector_PinHeader_2.54mm:PinHeader_1x03_P2.54mm_Vertical, symbol Connector:Conn_01x03_Male
- added J2: Comm, Connector_PinHeader_2.54mm:PinHeader_1x11_P2.54mm_Vertical, symbol Connector:Conn_01x11_Male
- added J3: CommLA, Connector_PinHeader_2.54mm:PinHeader_1x11_P2.54mm_Vertical, symbol Connector:Conn_01x11_Male
- added J4: PowerMon, Connector_PinHeader_2.54mm:PinHeader_1x05_P2.54mm_Vertical, symbol Connector:Conn_01x05_Male
- added J6: SWD0, Connector_PinHeader_2.54mm:PinHeader_1x03_P2.54mm_Vertical, symbol Connector:Conn_01x03_Male
- added J9: SWD1, Connector_PinHeader_2.54mm:PinHeader_1x03_P2.54mm_Vertical, symbol Connector:Conn_01x03_Male
- added JP1: Power source, Connector_PinHeader_2.54mm:PinHeader_1x03_P2.54mm_Vertical, symbol Jumper:Jumper_3_Bridged12
- added R1, R2, R3, R4, R5: 10k, Resistor_SMD:R_1206_3216Metric_Pad1.42x1.75mm_HandSolder, symbol Device:R_Small
- C1, C2: footprint (none) -> Capacitor_Tantalum_SMD:CP_EIA-3216-18_Kemet-A_Pad1.58x1.35mm_HandSolder
- J1: renamed from J13; footprint (none) -> Connector_USB:USB_Micro-B_Molex-105017-0001
- J10: renamed from J3; footprint (none) -> Connector_PinSocket_2.54mm:PinSocket_2x05_P2.54mm_Vertical
- J11: renamed from J8; value Target1 -> USB1; footprint (none) -> Connector_PinHeader_2.54mm:PinHeader_1x03_P2.54mm_Vertical
- J13: renamed from J4; footprint (none) -> Connector_PinSocket_2.54mm:PinSocket_2x05_P2.54mm_Vertical
- J14: renamed from J9; value Target1 -> USB2; footprint (none) -> Connector_PinHeader_2.54mm:PinHeader_1x03_P2.54mm_Vertical
- J16: renamed from J5; footprint (none) -> Connector_PinSocket_2.54mm:PinSocket_2x05_P2.54mm_Vertical
- J17: renamed from J10; value Target1 -> USB3; footprint (none) -> Connector_PinHeader_2.54mm:PinHeader_1x03_P2.54mm_Vertical
- J5: renamed from J6; footprint (none) -> Connector_PinHeader_2.54mm:PinHeader_1x03_P2.54mm_Vertical
- J7: renamed from J2; footprint (none) -> Connector_PinSocket_2.54mm:PinSocket_2x05_P2.54mm_Vertical
- J8: renamed from J7; value Target0 -> USB0; footprint (none) -> Connector_PinHeader_2.54mm:PinHeader_1x03_P2.54mm_Vertical
- U1: footprint (none) -> Package_TO_SOT_SMD:SOT-223-3_TabPin2
- U5: renamed from U8; footprint (none) -> Package_SO:SOIC-24W_7.5x15.4mm_P1.27mm
- renumbered U5 to U4, U4 to U6, U6 to U7
Connections:
- net MUXEN is gone; now on net GND: U4.15 (~E)
- net +3V3: now also J4.4 (Pin_4), R1.2, R3.1, R4.1
- net GND: now also J12.1 (Pin_1), J15.1 (Pin_1), J2.1 (Pin_1), J3.1 (Pin_1), J4.5 (Pin_5), J6.1 (Pin_1), J9.1 (Pin_1), R2.2, R5.2
- net PWR_EN: now also J2.10 (Pin_10), J3.10 (Pin_10), J4.3 (Pin_3), R5.1
- net SEL0: now also J2.6 (Pin_6), J3.6 (Pin_6)
- net SEL1: now also J2.7 (Pin_7), J3.7 (Pin_7)
- net T0_SWDIO: now also J6.3 (Pin_3)
- net T1_SWDIO: now also J9.3 (Pin_3)
- net T2_SWDIO: now also J12.3 (Pin_3)
- net T3_SWDIO: now also J15.3 (Pin_3)
- net T_BOOT0: now also J2.2 (Pin_2), J3.2 (Pin_2), R1.1
- net T_NRST: now also J2.3 (Pin_3), J3.3 (Pin_3), R2.1
- net T_RX: now also J2.5 (Pin_5), J3.5 (Pin_5)
- net T_TX: now also J2.4 (Pin_4), J3.4 (Pin_4)
- net T_VCC: now also J4.1 (Pin_1)
- net USBMUXEN0: now also J2.8 (Pin_8), J3.8 (Pin_8), R3.2
- net USBMUXEN1: now also J2.9 (Pin_9), J3.9 (Pin_9), R4.2
- net VBUS: now also JP1.1 (A); no longer C1.1, U1.3 (VI)
- net PWR_FAULT: now reaches U2.3 (FAULT)
- net PWR_FAULT: now also J4.2 (Pin_2)
- removed net SWCLK: J10.10 (Pin_10), J13.10 (Pin_10), J16.10 (Pin_10), J7.10 (Pin_10)
- new net: C1.1, JP1.2 (C), U1.3 (VI)
- new net EXT_5V: J2.11 (Pin_11), J3.11 (Pin_11), JP1.3 (B)
- new net T0_SWCLK: J6.2 (Pin_2), J7.10 (Pin_10)
- new net T1_SWCLK: J10.10 (Pin_10), J9.2 (Pin_2)
- new net T2_SWCLK: J12.2 (Pin_2), J13.10 (Pin_10)
- new net T3_SWCLK: J15.2 (Pin_2), J16.10 (Pin_10)
- no-connect marks 46 -> 25
Other:
- moved on the sheet: J1, J10, J11, J13, J14, J16, J17, J5, J8, U3, U5
